File: Dashboard PCB.kicad_pcb (KiCad board)
At the start: 2 copper layers, 200 x 100 mm, 62 parts, among them J1 Controls_Leader_Export_02x06, J2 CAN, J3 INDICATOR_SWITCH_OUT, J4 FAN_CTRL_01x02, J5 Horn_In_01x02, J6 Horn_Out_01x02, J7 CAN

Commit message: Routing finished :0
Parts:
- turned C8 to -90 degrees
- turned R8 to -90 degrees
Routing:
- net /LFT_OUT: track 0.00 -> 320.8 mm
- net /RT_OUT: track 0.00 -> 296.0 mm
- net /BPS_HZD: track 0.00 -> 278.8 mm
- net /CRUZ_SET: track 0.00 -> 274.2 mm
- net /IGN_ARR: track 0.00 -> 232.0 mm
- net /IGN_PWR: track 0.00 -> 195.6 mm
- net /CRUZ_EN: track 0.00 -> 184.1 mm
- net /FWD_SW: track 0.00 -> 177.7 mm
- net /REV_SW: track 0.00 -> 134.6 mm
- net /FAN+: track 0.00 -> 26.7 mm
- net Net-(D1-A): track 0.00 -> 24.9 mm
- net /FAN-: track 0.00 -> 22.2 mm
- net /CANGND: track 0.00 -> 17.8 mm
- net /CAN+12V: track 0.00 -> 17.8 mm
- net /CAN-H: track 0.00 -> 16.5 mm
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- added copper zone on F.Cu, net +12V
- added copper zone on B.Cu, net GND
