File: Dashboard PCB.kicad_pcb (KiCad board)
At the start: 2 copper layers, 150 x 100.2 mm, 66 parts, among them J1 Controls_Leader_Export_02x06, J2 Conn_02x03_CAN, J3 INDICATOR_SWITCH_OUT, J4 FAN_CTRL_01x02, J5 Horn_In_01x02, J6 Horn_Out_01x02, J7 Conn_02x03_CAN, J8 Supp_Out, J9 Supp_In

Commit message: Update Dashboard PCB.kicad_pcb
Routing:
- net /DBG_LED: track 106.0 -> 106.8 mm
- net /IGN_ARR: track 113.4 -> 113.5 mm, vias 1 -> 3
Changed lines of the file:
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@@
 		(tags "resistor")
 		(property "Reference" "R13"
-			(at 0 2 360)
+			(at 0 2 0)
 			(layer "B.SilkS")
 			(effects
@@
 		)
 		(property "Value" "HZD_RES_VAL"
-			(at 0 -1.65 360)
+			(at 0 -1.65 0)
 			(layer "B.Fab")
 			(effects
@@
 		)
 		(fp_text user "${REFERENCE}"
-			(at 0 -1 360)
+			(at 0 -1 0)
 			(layer "B.Fab")
 			(effects
@@
 	)
 	(segment
+		(start 150.8 62.8)
+		(end 143.8 62.8)
+		(width 0.25)
+		(layer "F.Cu")
+		(net 8)
+	)
+	(segment
 		(start 94.798508 68.0875)
 		(end 93.298508 69.5875)
@@
 	)
 	(segment
+		(start 174.74 89.34)
+		(end 174.6 89.2)
+		(width 0.25)
+		(layer "F.Cu")
+		(net 8)
+	)
+	(segment
+		(start 169.4 84)
+		(end 169.4 81.4)
+		(width 0.25)
+		(layer "F.Cu")
+		(net 8)
+	)
+	(segment
+		(start 169.4 81.4)
+		(end 150.8 62.8)
+		(width 0.25)
+		(layer "F.Cu")
+		(net 8)
+	)
+	(segment
 		(start 100.123508 68.0875)
 		(end 94.798508 68.0875)
@@
 		(net 8)
 	)
+	(segment
+		(start 174.6 89.2)
+		(end 169.4 84)
+		(width 0.25)
+		(layer "F.Cu")
+		(net 8)
+	)
+	(segment
+		(start 174.74 93.500018)
+		(end 174.74 89.34)
+		(width 0.25)
+		(layer "F.Cu")
+		(net 8)
+	)
+	(segment
+		(start 143.8 62.8)
+		(end 119 62.8)
+		(width 0.25)
+		(layer "F.Cu")
+		(net 8)
+	)
+	(via
+		(at 114.048508 62.8375)
+		(size 0.6)
+		(drill 0.3)
+		(layers "F.Cu" "B.Cu")
+		(net 8)
+	)
 	(via
 		(at 100.123508 68.0875)
@@
 		(net 8)
 	)
-	(segment
-		(start 169.4 84.04)
-		(end 169.4 81.4)
-		(width 0.25)
-		(layer "B.Cu")
+	(via
+		(at 119 62.8)
+		(size 0.6)
+		(drill 0.3)
+		(layers "F.Cu" "B.Cu")
 		(net 8)
 	)
@@
 	)
 	(segment
-		(start 169.4 81.4)
-		(end 150.8375 62.8375)
-		(width 0.25)
-		(layer "B.Cu")
-		(net 8)
-	)
-	(segment
 		(start 177.5 98.39)
 		(end 180.25 98.39)
@@
 	)
 	(segment
-		(start 174.74 93.500018)
-		(end 174.74 89.38)
-		(width 0.25)
-		(layer "B.Cu")
-		(net 8)
-	)
-	(segment
 		(start 114.048508 62.8375)
 		(end 108.798508 68.0875)
@@
 	)
 	(segment
-		(start 174.74 89.38)
-		(end 169.4 84.04)
+		(start 108.798508 68.0875)
+		(end 100.123508 68.0875)
 		(width 0.25)
 		(layer "B.Cu")
@@
 	)
 	(segment
-		(start 108.798508 68.0875)
-		(end 100.123508 68.0875)
+		(start 175.55 98.44)
+		(end 174.74 97.63)
 		(width 0.25)
 		(layer "B.Cu")
@@
 	)
 	(segment
-		(start 175.55 98.44)
-		(end 174.74 97.63)
+		(start 114.086008 62.8)
+		(end 114.048508 62.8375)
 		(width 0.25)
 		(layer "B.Cu")
@@
 	)
 	(segment
-		(start 150.8375 62.8375)
-		(end 114.048508 62.8375)
+		(start 119 62.8)
+		(end 114.086008 62.8)
 		(width 0.25)
 		(layer "B.Cu")
@@
 	)
 	(segment
-		(start 116.45 62.8)
-		(end 190.55 62.8)
+		(start 103.6625 75.5875)
+		(end 117.45 61.8)
 		(width 0.25)
 		(layer "F.Cu")
@@
 	)
 	(segment
-		(start 191.65 63.9)
-		(end 193.298508 63.9)
+		(start 189.55 61.8)
+		(end 191.65 63.9)
 		(width 0.25)
 		(layer "F.Cu")
@@
 	)
 	(segment
-		(start 103.6625 75.5875)
-		(end 116.45 62.8)
+		(start 191.65 63.9)
+		(end 193.298508 63.9)
 		(width 0.25)
 		(layer "F.Cu")
@@
 	)
 	(segment
-		(start 190.55 62.8)
-		(end 191.65 63.9)
+		(start 117.45 61.8)
+		(end 189.55 61.8)
 		(width 0.25)
 		(layer "F.Cu")

Commit message: Final changes for now
added p/n n stuff
Parts:
- renumbered HZD_SW1 to HZD_SW
Routing:
- net /IGN_ARR: vias 3 -> 2
Other:
- outline, holes or cut-outs redrawn
Changed lines of the file:
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@@
 		(layer "F.Cu")
 		(at 137.048508 85.3375)
-		(property "Reference" "HZD_SW1"
+		(property "Reference" "HZD_SW"
 			(at -0.16 7 0)
 			(unlocked yes)
@@
 		)
 	)
-	(gr_rect
-		(start 211.25 86.5)
-		(end 227.25 114.75)
+	(gr_line
+		(start 211.25533 87.25533)
+		(end 211.25033 113.99967)
 		(stroke
-			(width 0.1)
+			(width 0.05)
+			(type default)
+		)
+		(layer "Edge.Cuts")
+	)
+	(gr_arc
+		(start 226.49467 86.50533)
+		(mid 227.025 86.725)
+		(end 227.24467 87.25533)
+		(stroke
+			(width 0.05)
+			(type default)
+		)
+		(layer "Edge.Cuts")
+	)
+	(gr_arc
+		(start 227.25 114)
+		(mid 227.03033 114.53033)
+		(end 226.5 114.75)
+		(stroke
+			(width 0.05)
 			(type default)
 		)
-		(fill none)
 		(layer "Edge.Cuts")
 	)
@@
 		(layer "Edge.Cuts")
 	)
+	(gr_line
+		(start 226.49467 86.50533)
+		(end 212.00533 86.50533)
+		(stroke
+			(width 0.05)
+			(type default)
+		)
+		(layer "Edge.Cuts")
+	)
+	(gr_arc
+		(start 212.00033 114.74967)
+		(mid 211.47 114.53)
+		(end 211.25033 113.99967)
+		(stroke
+			(width 0.05)
+			(type default)
+		)
+		(layer "Edge.Cuts")
+	)
 	(gr_arc
 		(start 231.5 50.5875)
@@
 	)
 	(gr_arc
+		(start 211.25533 87.25533)
+		(mid 211.475 86.725)
+		(end 212.00533 86.50533)
+		(stroke
+			(width 0.05)
+			(type default)
+		)
+		(layer "Edge.Cuts")
+	)
+	(gr_line
+		(start 227.25 114)
+		(end 227.24467 87.25533)
+		(stroke
+			(width 0.05)
+			(type default)
+		)
+		(layer "Edge.Cuts")
+	)
+	(gr_arc
 		(start 83.548508 52.3375)
 		(mid 84.134294 50.923286)
@@
 	)
 	(gr_line
+		(start 212.00033 114.74967)
+		(end 226.5 114.75)
+		(stroke
+			(width 0.05)
+			(type default)
+		)
+		(layer "Edge.Cuts")
+	)
+	(gr_line
 		(start 233.5 148.5875)
 		(end 233.5 52.5875)
@@
 	)
 	(segment
-		(start 102.348508 130.3375)
-		(end 102.348508 128.7875)
+		(start 107.798508 79.5875)
+		(end 107.798508 79.018004)
 		(width 0.25)
 		(layer "B.Cu")
@@
 	)
 	(segment
-		(start 107.798508 79.5875)
-		(end 107.798508 78.8375)
+		(start 102.348508 130.3375)
+		(end 102.348508 128.7875)
 		(width 0.25)
 		(layer "B.Cu")
@@
 	)
 	(segment
-		(start 102.348508 128.7875)
-		(end 107.798508 123.3375)
-		(width 0.25)
-		(layer "B.Cu")
-		(net 4)
-	)
-	(segment
-		(start 106.548508 77.5875)
+		(start 106.368004 77.5875)
 		(end 106.048508 77.5875)
 		(width 0.25)
@@
 	)
 	(segment
-		(start 107.798508 78.8375)
-		(end 106.548508 77.5875)
+		(start 102.348508 128.7875)
+		(end 107.798508 123.3375)
 		(width 0.25)
 		(layer "B.Cu")
@@
 	)
 	(segment
+		(start 107.798508 79.018004)
+		(end 106.368004 77.5875)
+		(width 0.25)
+		(layer "B.Cu")
+		(net 4)
+	)
+	(segment
 		(start 109.25 87.788992)
 		(end 109.298508 87.8375)
@@
 		(net 8)
 	)
-	(via
-		(at 114.048508 62.8375)
-		(size 0.6)
-		(drill 0.3)
-		(layers "F.Cu" "B.Cu")
-		(net 8)
-	)
