File: hardware/ControlsLeader_PCB/ControlsLeader_PCB.kicad_pcb (KiCad board)
At the start: 2 copper layers, 135 x 72 mm, 173 parts, among them J1 CarCANConnector_Out, J11 EStop1, J12 SteeringConn_01x07, J13 Supp_Out, J15 IgnConn_01x04, J17 Conn_01x02, J2 PeripheralCAN_out, J3 CarCANConnector_In, J4 PeripheralCAN_in, J6 Conn_2Rows-13Pins, J7 Conn_01x04, J8 Dash_Lsom_Horn_Lights_PWR, J9 Supp_In, Q1 NMOS, Q10 NMOS, Q11 NMOS, Q12 NMOS, Q13 NMOS, Q14 NMOS, Q15 NMOS, Q16 NMOS, Q3 NMOS, Q4 NMOS, Q5 NMOS, Q6 NMOS, Q7 NMOS, Q8 NMOS, Q9 NMOS, U2 LeaderSOM, U4 LT1963AEST-3.3#TRPBF, U6 TPS5405DR

Commit message: ShaqDash is born. . . RPP in progress
Parts:
- removed 3.3V1, Cruise_En, Cruise_Set, FWD_SW, Hazard, Horn_In, Ign_OFF, Ign_arr, Ign_mtr, Left_Blinker, Neutral_gear, Regen_Active, Regen_En, Rev_SW, Right_Blinker: TestPoint, TestPoint:TestPoint_Pad_1.0x1.0mm
- removed Buck Status: Controls_Leader_Status_Red, LED_SMD:LED_0603_1608Metric_Pad1.05x0.95mm_HandSolder
- removed C35, C36: 10uF, Capacitor_SMD:C_0603_1608Metric_Pad1.08x0.95mm_HandSolder
- removed Cruise_En__Sig, Cruise_Set_Sig, FWD_SW_Sig, Horn_3.3V_Sig, Hzard_Sig, Left_Blinker_Sig, Neutral_Gear_Sig, Regen_Active_Sig, Regen_En_Sig, Rev_SW_Sig, Right_Blinker_Sig: GPIO_Status_Blue, LED_SMD:LED_0603_1608Metric_Pad1.05x0.95mm_HandSolder
- removed F1: Fuse, Fuse:Fuseholder_Blade_Mini_Keystone_3568
- removed the G*** at (119.2, 62.8)
- removed the G*** at (118.3, 83.4)
- removed J12: SteeringConn_01x07, Connector_Molex:Molex_Nano-Fit_105313-xx07_1x07_P2.50mm_Horizontal
- removed LDO Status: Controls_Leader_Status_Red, LED_SMD:LED_0603_1608Metric_Pad1.05x0.95mm_HandSolder
- removed U4: LT1963AEST-3.3#TRPBF, Package_TO_SOT_SMD:SOT-223-3_TabPin2
- added C19: .1u, Capacitor_SMD:C_0603_1608Metric_Pad1.08x0.95mm_HandSolder, F.Cu at (205.2, 82.1)
- added C20: 220n, Capacitor_SMD:C_0603_1608Metric_Pad1.08x0.95mm_HandSolder, F.Cu at (200.4, 87.2)
- added C21: 1u, Capacitor_SMD:C_0603_1608Metric_Pad1.08x0.95mm_HandSolder, F.Cu at (198.8, 84.0)
- added C22: 10u, Capacitor_SMD:C_0603_1608Metric_Pad1.08x0.95mm_HandSolder, F.Cu at (195.6, 80.2)
- added D1: GPIO_Status_Blue, LED_SMD:LED_0603_1608Metric_Pad1.05x0.95mm_HandSolder, F.Cu at (101.2, 114.8)
- added D10: GPIO_Status_Blue, LED_SMD:LED_0603_1608Metric_Pad1.05x0.95mm_HandSolder, F.Cu at (101.8, 101.2)
- added D11: GPIO_Status_Blue, LED_SMD:LED_0603_1608Metric_Pad1.05x0.95mm_HandSolder, F.Cu at (102.0, 88.9)
- added D12: GPIO_Status_Blue, LED_SMD:LED_0603_1608Metric_Pad1.05x0.95mm_HandSolder, F.Cu at (102.0, 104.0)
- added D13: GPIO_Status_Blue, LED_SMD:LED_0603_1608Metric_Pad1.05x0.95mm_HandSolder, F.Cu at (104.0, 114.8)
- added D14: GPIO_Status_Blue, LED_SMD:LED_0603_1608Metric_Pad1.05x0.95mm_HandSolder, F.Cu at (106.7, 114.8)
- added D15: GPIO_Status_Blue, LED_SMD:LED_0603_1608Metric_Pad1.05x0.95mm_HandSolder, F.Cu at (108.9, 114.7)
- added D2: GPIO_Status_Blue, LED_SMD:LED_0603_1608Metric_Pad1.05x0.95mm_HandSolder, F.Cu at (101.8, 85.6)
- added D28: Controls_Leader_Status_Red, LED_SMD:LED_0603_1608Metric_Pad1.05x0.95mm_HandSolder, F.Cu at (184.3, 70.4)
- added D3: GPIO_Status_Blue, LED_SMD:LED_0603_1608Metric_Pad1.05x0.95mm_HandSolder, F.Cu at (102.0, 92.2)
- added D5: GPIO_Status_Blue, LED_SMD:LED_0603_1608Metric_Pad1.05x0.95mm_HandSolder, F.Cu at (102.0, 97.8)
- added D9: GPIO_Status_Blue, LED_SMD:LED_0603_1608Metric_Pad1.05x0.95mm_HandSolder, F.Cu at (101.9, 95.2)
- added F3: Fuse, Fuse:Fuseholder_Blade_Mini_Keystone_3568, F.Cu at (195.5, 99.4)
- added J14: SteeringConn_01x06, Connector_Molex:Molex_Nano-Fit_105313-xx06_1x06_P2.50mm_Horizontal, F.Cu at (109.2, 118.8)
- added R58: 200k, Resistor_SMD:R_0603_1608Metric_Pad0.98x0.95mm_HandSolder, F.Cu at (204.8, 84.7)
- added R59: 9k, Resistor_SMD:R_0603_1608Metric_Pad0.98x0.95mm_HandSolder, F.Cu at (201.3, 82.1)
- added RPP1: LM74502HDDFR, UTSVT_Power:SOT65P280X110-8N, F.Cu at (201.8, 84.7)
- added TP1: TestPoint, TestPoint:TestPoint_Pad_1.0x1.0mm, F.Cu at (116.0, 106.5)
- added TP10: TestPoint, TestPoint:TestPoint_Pad_1.0x1.0mm, F.Cu at (153.9, 84.5)
- added TP11: TestPoint, TestPoint:TestPoint_Pad_1.0x1.0mm, F.Cu at (116.0, 101.6)
- added TP12: TestPoint, TestPoint:TestPoint_Pad_1.0x1.0mm, F.Cu at (116.0, 110.8)
- added TP13: TestPoint, TestPoint:TestPoint_Pad_1.0x1.0mm, F.Cu at (116.0, 115.3)
- added TP15: TestPoint, TestPoint:TestPoint_Pad_1.0x1.0mm, F.Cu at (116.0, 120.2)
- added TP2: TestPoint, TestPoint:TestPoint_Pad_1.0x1.0mm, F.Cu at (161.0, 84.4)
- added TP3: TestPoint, TestPoint:TestPoint_Pad_1.0x1.0mm, F.Cu at (148.2, 84.5)
- added TP4: TestPoint, TestPoint:TestPoint_Pad_1.0x1.0mm, F.Cu at (142.3, 84.5)
- added TP5: TestPoint, TestPoint:TestPoint_Pad_1.0x1.0mm, F.Cu at (179.2, 103.0)
- added TP6: TestPoint, TestPoint:TestPoint_Pad_1.0x1.0mm, F.Cu at (177.7, 107.6)
- added TP7: TestPoint, TestPoint:TestPoint_Pad_1.0x1.0mm, F.Cu at (179.1, 95.2)
- added TP8: TestPoint, TestPoint:TestPoint_Pad_1.0x1.0mm, F.Cu at (136.5, 84.7)
- added TP9: TestPoint, TestPoint:TestPoint_Pad_1.0x1.0mm, F.Cu at (116.0, 96.8)
- D29: footprint Diode_SMD:D_SOD-523 -> Diode_SMD:D_SOD-123F
- R1, R10, R11, R12, R13, R14, R15, R16, R17, R18, R19, R2, R20, R21, R22, R23, R24, R25, R26, R27, R28, R29, R3, R30, R31, R32, R34, R35, R36, R37, R38, R39, R4, R40, R41, R42, R43, R44, R47, R5, R57, R6, R7, R8, R9: footprint Capacitor_SMD:C_0603_1608Metric_Pad1.08x0.95mm_HandSolder -> Resistor_SMD:R_0603_1608Metric_Pad0.98x0.95mm_HandSolder
- R33, R45, R46, R55: value 65 -> 120; footprint Capacitor_SMD:C_0603_1608Metric_Pad1.08x0.95mm_HandSolder -> Resistor_SMD:R_0603_1608Metric_Pad0.98x0.95mm_HandSolder
- R48, R49, R50, R51, R52, R53, R54: value 20 -> 120; footprint Capacitor_SMD:C_0603_1608Metric_Pad1.08x0.95mm_HandSolder -> Resistor_SMD:R_0603_1608Metric_Pad0.98x0.95mm_HandSolder
- R56: value 1.1k -> 10k; footprint Capacitor_SMD:C_0603_1608Metric_Pad1.08x0.95mm_HandSolder -> Resistor_SMD:R_0603_1608Metric_Pad0.98x0.95mm_HandSolder
- moved G*** 82.0 mm to (118.4, 69.8)
- moved R56 78.5 mm to (203.9, 87.2), turned to 180 degrees
- moved J2 3.34 mm to (128.5, 69.0)
- moved J4 3.34 mm to (141.5, 69.0)
- moved J15 2.91 mm to (157.1, 69.0)
- moved D6 2.73 mm to (162.3, 72.7)
- moved D7 2.73 mm to (166.9, 72.7)
- moved D8 2.73 mm to (159.4, 72.5)
- moved R21 2.73 mm to (162.2, 76.1)
- moved R22 2.73 mm to (166.9, 76.2)
- moved R23 2.73 mm to (159.4, 76.1)
- moved C15 1.97 mm to (193.1, 81.0)
- moved C16 1.97 mm to (194.0, 78.6)
- moved C17 1.97 mm to (191.5, 73.7)
- moved C18 1.97 mm to (187.5, 73.4)
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Connections:
- net /Horn_3.3V_Signal renamed /Horn_5V_Signal
- F2 pad 1: Net-(Q6-D) -> /+24v_Horn
- F2 pad 2: /Horn_24V_Signal_Out -> Net-(J8-Pin_3)
- J15 pad 1: /3.3V_LDO -> /5V_LDO
- J6 pad 1: /3.3V_LDO -> /5V_LDO
- J6 pad 3: /3.3V_LDO -> /5V_LDO
- J6 pad 5: /3.3V_LDO -> /5V_LDO
- J6 pad 7: /3.3V_LDO -> /5V_LDO
- J6 pad 9: /3.3V_LDO -> /5V_LDO
- J8 pad 1: +24V -> /RPP/LV+
- J8 pad 2: /+24v_Lights -> Net-(J8-Pin_2)
- J8 pad 3: /+24v_Horn -> Net-(J8-Pin_3)
- Q6 pad 1: Net-(Q6-D) -> /Horn_24V_Signal_Out
- R48 pad 1: Net-(D19-K) -> Net-(D27-K)
- R49 pad 1: Net-(D20-K) -> GND
- R49 pad 2: GND -> Net-(D19-K)
- R50 pad 1: Net-(D21-K) -> GND
- R50 pad 2: GND -> Net-(D20-K)
- R51 pad 1: Net-(D22-K) -> Net-(D21-K)
- R52 pad 1: Net-(D23-K) -> Net-(D22-K)
- R53 pad 1: Net-(D24-K) -> Net-(D23-K)
- R54 pad 1: Net-(D25-K) -> Net-(D24-K)
- R55 pad 1: Net-(D27-K) -> Net-(D25-K)
- R56 pad 1: Net-(D30-K) -> /RPP/LV+
- R56 pad 2: GND -> /RPP/RPP_EN
- U2 pad 38: GND -> unconnected-(U2B-GNDA-Pad38)
Routing:
- net /3.3V_LDO: track 144.6 -> 0.00 mm, vias 1 -> 0
- net Net-(Q6-D): track 30.8 -> 0.00 mm, vias 1 -> 0
- net /5V_LDO: track 132.4 -> 153.7 mm, vias 5 -> 6
- net /5v_3.3v_LDO/3.3V_LDO: track 20.4 -> 0.00 mm, vias 2 -> 0
- net /+24v_Horn: track 22.2 -> 41.6 mm
- net Net-(J8-Pin_3): track 0.00 -> 18.5 mm
- net Net-(J8-Pin_2): track 0.00 -> 14.4 mm
- net /+24v_Lights: track 87.5 -> 73.9 mm
- net GND: track 139.4 -> 126.1 mm, vias 41 -> 155
- net /RPP/LV+: track 0.00 -> 12.9 mm, vias 0 -> 1
- net Net-(D30-K): track 7.95 -> 0.00 mm
- net /RPP/RPP_EN: track 0.00 -> 5.91 mm
- net Net-(RPP1-OV): track 0.00 -> 5.22 mm
- net +24V: track 149.8 -> 153.4 mm
- net /3.3V_LSOM: track 130.5 -> 127.3 mm
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- added copper zone on F.Cu, net /RPP/RPP_EN
Other:
- board text added: "Buck Status"
- board text added: "Cruise_En"
- board text added: "Cruise_En__Sig"
- board text added: "Cruise_Set"
- board text added: "Cruise_Set_Sig"
- board text added: "E Stop"
- board text added: "FWD_SW"
- board text added: "FWD_SW_Sig"
- board text added: "Hazard"
- board text added: "Horn_3.3V_Sig"
- board text added: "Horn_In"
- board text added: "Hzard_Sig"
- board text added: "Ign_OFF"
- board text added: "Ign_arr"
- board text added: "Ign_mtr"
- board text added: "Left_Blinker"
- board text added: "Left_Blinker_Sig"
- board text added: "Neutral_gear"
- board text added: "Regen_Active"
- board text added: "Regen_Active_Sig"
- board text added: "Regen_En"
- board text added: "Regen_En_Sig"
- board text added: "Rev_SW"
- board text added: "Rev_SW_Sig"
- board text added: "Right_Blinker"
- board text added: "Right_Blinker_Sig"
- board text removed: "E-Stop"

Commit message: Rev B :)
Parts:
- added D30: SMAF4758A, UTSVT_Passives:SODFL5026X125N, F.Cu at (196.2, 81.7)
- added Q17: NVMFWS1D7N04XMT1G, NVMFWS3D0P04M8LT1G:NVMFWS3D0P04M8LT1G, F.Cu at (198.3, 63.7)
- added Q2: NVMFWS1D7N04XMT1G, NVMFWS3D0P04M8LT1G:NVMFWS3D0P04M8LT1G, F.Cu at (207.0, 63.7)
- moved R55 20.2 mm to (181.9, 119.5)
- moved G*** 10.5 mm to (120.6, 80.1)
- moved J13 9.20 mm to (189.2, 69.0)
- moved J9 9.20 mm to (181.2, 69.0)
- moved C32 9.10 mm to (172.7, 70.2)
- moved D28 9.10 mm to (175.2, 71.1)
- moved C33 9.10 mm to (169.7, 70.2)
- moved C34 9.10 mm to (167.7, 70.2)
- moved R54 5.78 mm to (187.7, 119.4)
- moved R52 5.76 mm to (190.6, 119.3)
- moved D6 5.67 mm to (156.6, 72.6)
- moved D7 5.67 mm to (161.2, 72.6)
- moved D8 5.67 mm to (153.7, 72.5)
- moved R22 5.67 mm to (161.2, 76.2)
- moved R23 5.67 mm to (153.7, 76.1)
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Connections:
- RPP1 pad 8: Net-(RPP1-SRC) -> /RPP/NVM_Lbl
Routing:
- net Net-(RPP1-GATE): track 0.00 -> 31.1 mm
- net +24V: track 153.4 -> 176.8 mm
- net /RPP/NVM_Lbl: track 0.00 -> 21.0 mm
- net /RPP/LV+: track 12.9 -> 33.0 mm
- net /PerCan_L: track 75.7 -> 82.6 mm, vias 4 -> 3
- net /+24v_Lights: track 73.9 -> 80.6 mm
- net /Ign_mtr_Signal: track 38.5 -> 45.1 mm
- net GND: track 126.1 -> 119.8 mm, vias 155 -> 174
- net /PerCan_H: track 84.1 -> 89.9 mm
- net /5V_LDO: track 153.7 -> 148.3 mm
- net /Ign_off_Signal: track 46.9 -> 51.6 mm
- net /RPP/RPP_EN: track 5.91 -> 8.88 mm
- net Net-(D28-K): track 2.67 -> 5.30 mm
- net /Ign_arr_Signal: track 56.2 -> 58.6 mm
- net /Dash/LV-: track 10.1 -> 9.42 mm
- added copper zone on F.Cu, net /RPP/NVM_Lbl
