File: hardware/ControlsLeader_PCB/ControlsLeader_PCB.kicad_pcb (KiCad board)
At the start: 2 copper layers, 135 x 72 mm, 176 parts, among them J1 CarCANConnector_Out, J11 EStop1, J13 Supp_Out, J14 SteeringConn_01x06, J15 IgnConn_01x04, J17 Conn_01x02, J2 PeripheralCAN_out, J3 CarCANConnector_In, J4 PeripheralCAN_in, J6 Conn_2Rows-13Pins, J7 Conn_01x04, J8 Dash_Lsom_Horn_Lights_PWR, J9 Supp_In, Q1 NMOS, Q10 NMOS, Q11 NMOS, Q12 NMOS, Q13 NMOS, Q14 NMOS, Q15 NMOS, Q16 NMOS, Q17 NVMFWS1D7N04XMT1G, Q2 NVMFWS1D7N04XMT1G, Q3 NMOS, Q4 NMOS, Q5 NMOS, Q6 NMOS, Q7 NMOS, Q8 NMOS, Q9 NMOS, U2 LeaderSOM, U6 TPS5405DR

Commit message: Steering Angle Sensor SCH changes
Parts:
- removed the G*** at (195.8, 96.5)
- added R60: 0, Resistor_SMD:R_0603_1608Metric_Pad0.98x0.95mm_HandSolder, B.Cu at (201.9, 95.2)
- added R61: 0, Resistor_SMD:R_0603_1608Metric_Pad0.98x0.95mm_HandSolder, B.Cu at (203.8, 95.2)
- moved J11 114.6 mm to (95.9, 89.5), turned to 180 degrees
- moved J7 112.9 mm to (95.9, 81.4), turned to 180 degrees
- moved G*** 14.9 mm to (153.4, 90.6)
- moved Q17 9.41 mm to (198.1, 73.1), turned to 180 degrees
- moved Q2 8.96 mm to (198.1, 64.4), turned to 0 degrees
- moved J6 3.06 mm to (98.4, 106.9)
- moved R59 0.94 mm to (200.6, 81.5)
- moved G*** 0.28 mm to (120.8, 80.1)
Connections:
- net /5V_LDO renamed /5V_Buck
- Q17 pad 1: +24V -> Net-(RPP1-SRC)
- Q17 pad 2: +24V -> Net-(RPP1-SRC)
- Q17 pad 3: +24V -> Net-(RPP1-SRC)
- Q17 pad 5: /RPP/NVM_Lbl -> +24V
- Q17 pad 6: /RPP/NVM_Lbl -> +24V
- Q17 pad 7: /RPP/NVM_Lbl -> +24V
- Q17 pad 8: /RPP/NVM_Lbl -> +24V
- Q17 pad 9: /RPP/NVM_Lbl -> +24V
- Q2 pad 1: /RPP/NVM_Lbl -> Net-(RPP1-SRC)
- Q2 pad 2: /RPP/NVM_Lbl -> Net-(RPP1-SRC)
- Q2 pad 3: /RPP/NVM_Lbl -> Net-(RPP1-SRC)
- RPP1 pad 8: /RPP/NVM_Lbl -> Net-(RPP1-SRC)
Routing:
- net Net-(RPP1-SRC): track 0.00 -> 27.2 mm
- net /RPP/NVM_Lbl: track 21.0 -> 0.00 mm
- net +24V: track 176.8 -> 167.7 mm, vias 3 -> 5
- net /5V_Buck: track 148.3 -> 141.9 mm
- net /Regen_Enable_Signal: track 66.7 -> 70.2 mm
- net Net-(J8-Pin_2): track 14.4 -> 17.2 mm
- net /+24v_Horn: track 41.6 -> 44.3 mm
- net /Fwd_SW_Signal: track 79.8 -> 82.4 mm
- net /Cruise_Enable_Signal: track 46.6 -> 48.8 mm
- net /Neutral_Gear_Signal: track 60.8 -> 62.8 mm
- net Net-(J8-Pin_3): track 18.5 -> 20.4 mm
- net /Cruise_Set_Signal: track 30.0 -> 31.8 mm
- net /RPP/LV+: track 33.0 -> 34.6 mm
- net /Rev_SW_Signal: track 56.5 -> 57.9 mm
- net /Horn_24V_Signal_Out: track 30.0 -> 28.7 mm
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- removed copper zone on F.Cu, net /RPP/NVM_Lbl
Other:
- board text added: "Horns_24v_short"
- board text added: "Lights_24v_short"

Commit message: revb layout, working on silkscreen
Parts:
- removed D26, D27: 0603_SMD, LED_SMD:LED_0603_1608Metric_Pad1.05x0.95mm_HandSolder
- removed R48: 120, Resistor_SMD:R_0603_1608Metric_Pad0.98x0.95mm_HandSolder
- added 16v_Out1: 5V_Out, TestPoint:TestPoint_Pad_1.0x1.0mm, B.Cu at (218.3, 117.5)
- added Adj16V1: Adj5V, TestPoint:TestPoint_Pad_1.0x1.0mm, B.Cu at (214.9, 120.1)
- added C23: 0.1uF, Capacitor_SMD:C_0603_1608Metric_Pad1.08x0.95mm_HandSolder, F.Cu at (185.2, 111.2)
- added C24: 1uF, Capacitor_SMD:C_0603_1608Metric_Pad1.08x0.95mm_HandSolder, F.Cu at (183.7, 111.2)
- added C25: 1uF, Capacitor_SMD:C_0603_1608Metric_Pad1.08x0.95mm_HandSolder, F.Cu at (209.9, 113.3)
- added C26: 10uF, Capacitor_SMD:C_0603_1608Metric_Pad1.08x0.95mm_HandSolder, F.Cu at (209.9, 116.8)
- added C27: 2.2uF, Capacitor_SMD:C_0603_1608Metric_Pad1.08x0.95mm_HandSolder, F.Cu at (216.8, 113.1)
- added C28: 5uF, Capacitor_SMD:C_0603_1608Metric_Pad1.08x0.95mm_HandSolder, F.Cu at (205.3, 121.8)
- added CC_FLT1: LED, LED_SMD:LED_0603_1608Metric_Pad1.05x0.95mm_HandSolder, F.Cu at (184.1, 116.2)
- added CC_Term1: Jumper_2_Open, Connector_PinHeader_2.54mm:PinHeader_1x02_P2.54mm_Vertical, F.Cu at (196.2, 112.0)
- added En16V1: Enable5V, TestPoint:TestPoint_Pad_1.0x1.0mm, B.Cu at (205.6, 117.7)
- added F1: 0603L025YR, 0603L025YR:FUSC1608X75N, F.Cu at (218.4, 114.8)
- added F4: 0603L025YR, 0603L025YR:FUSC1608X75N, F.Cu at (192.1, 74.0)
- added F5: 0603L025YR, 0603L025YR:FUSC1608X75N, F.Cu at (100.3, 83.1)
- added IC1: TCAN337DCNR, UTSVT_ICs:TCAN337DCNR, F.Cu at (188.1, 112.1)
- added IC2: AP2205-W5-7, AP2205-W5-7:AP2205W57, F.Cu at (213.3, 115.0)
- added J12: SteeringAngleConn_01x04, Connector_Molex:Molex_Nano-Fit_105313-xx04_1x04_P2.50mm_Horizontal, F.Cu at (208.8, 79.2)
- added J16: Conn_01x03, Connector_Molex:Molex_Nano-Fit_105313-xx03_1x03_P2.50mm_Horizontal, F.Cu at (208.7, 69.0)
- added Q18: NMOS, LSOM_IRLM:SOT23, F.Cu at (201.8, 119.1)
- added R62: 10k, Resistor_SMD:R_0603_1608Metric_Pad0.98x0.95mm_HandSolder, F.Cu at (187.7, 114.7)
- added R63: 2.2k, Resistor_SMD:R_0603_1608Metric_Pad0.98x0.95mm_HandSolder, F.Cu at (187.7, 116.2)
- added R64: 10k, Resistor_SMD:R_0603_1608Metric_Pad0.98x0.95mm_HandSolder, F.Cu at (208.4, 115.1)
- added R65: 115k, Resistor_SMD:R_0603_1608Metric_Pad0.98x0.95mm_HandSolder, F.Cu at (216.8, 116.5)
- added R66: 10k, Resistor_SMD:R_0603_1608Metric_Pad0.98x0.95mm_HandSolder, F.Cu at (213.3, 118.4)
- added R67: 100k, Resistor_SMD:R_0603_1608Metric_Pad0.98x0.95mm_HandSolder, F.Cu at (204.2, 116.3)
- added R68: 120, Resistor_SMD:R_0603_1608Metric_Pad0.98x0.95mm_HandSolder, F.Cu at (194.5, 109.4)
- added TP14: TestPoint, TestPoint:TestPoint_Pad_1.0x1.0mm, F.Cu at (200.4, 115.9)
- added U1: CDSOT23-T24CAN, UTSVT_ICs:CDSOT23-T24CAN, F.Cu at (192.3, 112.0)
- added Vin1: Vin, TestPoint:TestPoint_Pad_1.0x1.0mm, B.Cu at (198.8, 113.8)
- D17: value 0603_SMD -> GPIO_Status_Blue
- Q6: value NMOS -> NVMFWS1D7N04XMT1G; footprint LSOM_IRLM:SOT23 -> NVMFWS3D0P04M8LT1G:NVMFWS3D0P04M8LT1G
- R45: value 120 -> 10k
- R46: value 120 -> 150
- moved D17 8.96 mm to (201.8, 121.8), turned to 90 degrees
- moved R45 7.59 mm to (203.6, 121.8)
- moved R46 5.46 mm to (202.7, 124.3), turned to 0 degrees
- moved Q6 4.60 mm to (188.3, 105.6)
- moved G*** 0.44 mm to (198.8, 127.8)
Connections:
- net Net-(RPP1-SRC) renamed /RPP/RPP1_SRC
- D17 pad 2: /Extra_LED1 -> /PTT_Signal
- J14 pad 5: /Indicator_PWM -> /PTT_Signal
- J14 pad 6: /5V_Buck -> /5V_Buck_SteeringDash
- J6 pad 1: /5V_Buck -> /5V_Buck_SteeringDash
- J6 pad 3: /5V_Buck -> /5V_Buck_SteeringDash
- J6 pad 5: /5V_Buck -> /5V_Buck_SteeringDash
- J6 pad 7: /5V_Buck -> /5V_Buck_SteeringDash
- J6 pad 9: /5V_Buck -> /5V_Buck_SteeringDash
- Q6 pad 1: /Horn_24V_Signal_Out -> GND
- Q6 pad 2: /Horn_GPIO_OUT -> GND
- R45 pad 1: Net-(D17-K) -> GND
- R45 pad 2: GND -> /PTT_Signal
- R46 pad 1: Net-(D26-K) -> Net-(D17-K)
- U2 pad 10: /Extra_LED4 -> /PTT_GPIO_IN
- U2 pad 12: /Extra_LED3 -> /FDCAN2_RX
- U2 pad 20: /Extra_LED1 -> /FDCAN2_TX
Routing:
- net /PTT_Signal: track 0.00 -> 116.7 mm
- net /Indicator_PWM: track 43.1 -> 132.3 mm, vias 0 -> 1
- net /PTT_GPIO_IN: track 0.00 -> 87.0 mm, vias 0 -> 2
- net /Extra_LED1: track 78.1 -> 0.00 mm, vias 2 -> 0
- net /Extra_LED3: track 68.3 -> 0.00 mm, vias 2 -> 0
- net /Extra_LED4: track 64.1 -> 0.00 mm, vias 2 -> 0
- net /Steering Angle Sensor Components/SteeringCAN_L: track 0.00 -> 59.6 mm, vias 0 -> 1
- net /FDCAN2_TX: track 0.00 -> 59.0 mm
- net /FDCAN2_RX: track 0.00 -> 53.4 mm, vias 0 -> 2
- net /5V_Buck_SteeringDash: track 0.00 -> 52.5 mm, vias 0 -> 1
- net /Steering Angle Sensor Components/SteeringCAN_H: track 0.00 -> 49.9 mm, vias 0 -> 1
- net /5V_Buck: track 141.9 -> 93.2 mm, vias 6 -> 8
- net /3.3V_LSOM: track 127.3 -> 170.5 mm, vias 15 -> 19
- net +16V: track 0.00 -> 33.4 mm
- net /Horn_24V_Signal_Out: track 28.7 -> 5.35 mm, vias 2 -> 9
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- added copper zone on B.Cu, net /Horn_24V_Signal_Out
- added copper zone on F.Cu, net /Horn_24V_Signal_Out
- added copper zone on F.Cu, net /RPP/RPP1_SRC
