File: hardware/ControlsLeader_PCB/NMOS_SW.kicad_sch (KiCad schematic)
At the start: 7 parts, among them Q1 NMOS

Commit message: Rev B Layout
Parts:
- C1: value 5uF -> 1uF
- R31: value 100k -> 10k
Changed lines of the file:
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@@
 			)
 		)
-		(property "Value" "5uF"
+		(property "Value" "1uF"
 			(at 124.206 103.378 0)
 			(effects
@@
 			)
 		)
-		(property "Value" "100k"
+		(property "Value" "10k"
 			(at 144.78 90.1699 0)
 			(effects
