File: hardware/ControlsLeader_PCB/NMOS_SW.kicad_sch (KiCad schematic)
At the start: 7 parts, among them Q1 NMOS

Commit message: Mika is quite smart (#12)
Parts:
- C1: value 5uF -> 2.2uF
Connections:
- net 3.3V_Switch_Signal renamed 5V_Switch_Signal
Changed lines of the file:
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@@
 		)
 	)
-	(hierarchical_label "3.3V_Switch_Signal"
+	(hierarchical_label "5V_Switch_Signal"
 		(shape input)
 		(at 118.11 100.33 180)
@@
 		(instances
 			(project "ControlsLeader_PCB"
+				(path "/298dad81-302c-41c7-874b-fcde1c3cde17/cf34858a-7a31-4837-b51d-ee9ae3dd074c/85edfe3f-5ae7-4090-bed8-3b0581e114ea"
+					(reference "#PWR078")
+					(unit 1)
+				)
 				(path "/298dad81-302c-41c7-874b-fcde1c3cde17/cf34858a-7a31-4837-b51d-ee9ae3dd074c/879fa84f-14ed-4d21-9f88-1baa6fbdbf33"
 					(reference "#PWR087")
@@
 		(instances
 			(project "ControlsLeader_PCB"
+				(path "/298dad81-302c-41c7-874b-fcde1c3cde17/cf34858a-7a31-4837-b51d-ee9ae3dd074c/85edfe3f-5ae7-4090-bed8-3b0581e114ea"
+					(reference "#PWR080")
+					(unit 1)
+				)
 				(path "/298dad81-302c-41c7-874b-fcde1c3cde17/cf34858a-7a31-4837-b51d-ee9ae3dd074c/879fa84f-14ed-4d21-9f88-1baa6fbdbf33"
 					(reference "#PWR024")
@@
 			)
 		)
-		(property "Value" "5uF"
+		(property "Value" "2.2uF"
 			(at 124.206 103.378 0)
 			(effects
@@
 		(instances
 			(project "ControlsLeader_PCB"
+				(path "/298dad81-302c-41c7-874b-fcde1c3cde17/cf34858a-7a31-4837-b51d-ee9ae3dd074c/85edfe3f-5ae7-4090-bed8-3b0581e114ea"
+					(reference "C28")
+					(unit 1)
+				)
 				(path "/298dad81-302c-41c7-874b-fcde1c3cde17/cf34858a-7a31-4837-b51d-ee9ae3dd074c/879fa84f-14ed-4d21-9f88-1baa6fbdbf33"
 					(reference "C13")
@@
 		(instances
 			(project "ControlsLeader_PCB"
+				(path "/298dad81-302c-41c7-874b-fcde1c3cde17/cf34858a-7a31-4837-b51d-ee9ae3dd074c/85edfe3f-5ae7-4090-bed8-3b0581e114ea"
+					(reference "R46")
+					(unit 1)
+				)
 				(path "/298dad81-302c-41c7-874b-fcde1c3cde17/cf34858a-7a31-4837-b51d-ee9ae3dd074c/879fa84f-14ed-4d21-9f88-1baa6fbdbf33"
 					(reference "R29")
@@
 		(instances
 			(project "ControlsLeader_PCB"
+				(path "/298dad81-302c-41c7-874b-fcde1c3cde17/cf34858a-7a31-4837-b51d-ee9ae3dd074c/85edfe3f-5ae7-4090-bed8-3b0581e114ea"
+					(reference "#PWR067")
+					(unit 1)
+				)
 				(path "/298dad81-302c-41c7-874b-fcde1c3cde17/cf34858a-7a31-4837-b51d-ee9ae3dd074c/879fa84f-14ed-4d21-9f88-1baa6fbdbf33"
 					(reference "#PWR023")
@@
 		(instances
 			(project "ControlsLeader_PCB"
+				(path "/298dad81-302c-41c7-874b-fcde1c3cde17/cf34858a-7a31-4837-b51d-ee9ae3dd074c/85edfe3f-5ae7-4090-bed8-3b0581e114ea"
+					(reference "Q18")
+					(unit 1)
+				)
 				(path "/298dad81-302c-41c7-874b-fcde1c3cde17/cf34858a-7a31-4837-b51d-ee9ae3dd074c/879fa84f-14ed-4d21-9f88-1baa6fbdbf33"
 					(reference "Q15")
@@
 		(instances
 			(project "ControlsLeader_PCB"
+				(path "/298dad81-302c-41c7-874b-fcde1c3cde17/cf34858a-7a31-4837-b51d-ee9ae3dd074c/85edfe3f-5ae7-4090-bed8-3b0581e114ea"
+					(reference "R45")
+					(unit 1)
+				)
 				(path "/298dad81-302c-41c7-874b-fcde1c3cde17/cf34858a-7a31-4837-b51d-ee9ae3dd074c/879fa84f-14ed-4d21-9f88-1baa6fbdbf33"
 					(reference "R16")
@@
 		(instances
 			(project "ControlsLeader_PCB"
+				(path "/298dad81-302c-41c7-874b-fcde1c3cde17/cf34858a-7a31-4837-b51d-ee9ae3dd074c/85edfe3f-5ae7-4090-bed8-3b0581e114ea"
+					(reference "TP14")
+					(unit 1)
+				)
 				(path "/298dad81-302c-41c7-874b-fcde1c3cde17/cf34858a-7a31-4837-b51d-ee9ae3dd074c/879fa84f-14ed-4d21-9f88-1baa6fbdbf33"
 					(reference "TP13")
@@
 		(dnp no)
 		(property "Reference" "D1"
-			(at 137.16 104.4574 90)
+			(at 134.874 104.394 90)
 			(effects
 				(font
@@
 		(instances
 			(project "ControlsLeader_PCB"
+				(path "/298dad81-302c-41c7-874b-fcde1c3cde17/cf34858a-7a31-4837-b51d-ee9ae3dd074c/85edfe3f-5ae7-4090-bed8-3b0581e114ea"
+					(reference "D17")
+					(unit 1)
+				)
 				(path "/298dad81-302c-41c7-874b-fcde1c3cde17/cf34858a-7a31-4837-b51d-ee9ae3dd074c/879fa84f-14ed-4d21-9f88-1baa6fbdbf33"
 					(reference "D14")
@@
 		(instances
 			(project "ControlsLeader_PCB"
+				(path "/298dad81-302c-41c7-874b-fcde1c3cde17/cf34858a-7a31-4837-b51d-ee9ae3dd074c/85edfe3f-5ae7-4090-bed8-3b0581e114ea"
+					(reference "R67")
+					(unit 1)
+				)
 				(path "/298dad81-302c-41c7-874b-fcde1c3cde17/cf34858a-7a31-4837-b51d-ee9ae3dd074c/879fa84f-14ed-4d21-9f88-1baa6fbdbf33"
 					(reference "R44")
