File: hardware/ControlsLeader_PCB/RPP.kicad_sch (KiCad schematic)
At the start: 11 parts, among them Q17 NMOS, Q2 NMOS

Commit message: Rev B :)
Parts:
- removed Q17, Q2: NMOS, symbol Simulation_SPICE:NMOS
- added Q17, Q2: NVMFWS1D7N04XMT1G, NVMFWS3D0P04M8LT1G:NVMFWS3D0P04M8LT1G, symbol NVMFWS1D7N04XMT1G:NVMFWS1D7N04XMT1G
- D30: value SMZxxx -> SMAF4758A; footprint Diode_SMD:D_MELF -> UTSVT_Passives:SODFL5026X125N; now fitted
Connections:
- net 24_out: now also Q17.1, Q17.2, Q17.3
- net 24v_Ext: now also Q2.5, Q2.6, Q2.7, Q2.8, Q2.9
- net at RPP1.6 (GATE): now also Q17.4, Q2.4
- net NVM_Lbl: now reaches RPP1.8 (SRC)
- net NVM_Lbl: now also Q17.5, Q17.6, Q17.7, Q17.8, Q17.9, Q2.1, Q2.2, Q2.3
Other:
- moved on the sheet: C22

Commit message: Steering Angle Sensor SCH changes
Connections:
- net 24_out: now also Q17.5, Q17.6, Q17.7, Q17.8, Q17.9; no longer Q17.1, Q17.2, Q17.3
- net NVM_Lbl: no longer Q17.5, Q17.6, Q17.7, Q17.8, Q17.9, Q2.1, Q2.2, Q2.3, RPP1.8 (SRC)
- new net: Q17.1, Q17.2, Q17.3, Q2.1, Q2.2, Q2.3, RPP1.8 (SRC)
Other:
- moved on the sheet: Q17

Commit message: revb layout, working on silkscreen
Connections:
- net RPP1_SRC: now reaches Q17.1, Q17.2, Q17.3, Q2.1, Q2.2, Q2.3, RPP1.8 (SRC)
Changed lines of the file:
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@@
+		)
+	)
+	(label "RPP1_SRC"
+		(at 154.94 90.678 90)
+		(effects
+			(font
+				(size 1.27 1.27)
+			)
+			(justify left bottom)
 		)
 	)
