File: hardware/ControlsLeader_PCB/SteerinAngle.kicad_sch (KiCad schematic)
At the start: 1 part, among them J12 SteeringAngleConn_01x04

Commit message: revb layout, working on silkscreen
Connections:
- net FDCAN1_RX renamed SteeringCAN_L
- net FDCAN1_TX renamed SteeringCAN_H
Other:
- sheet 24v to 16v ldo ports: added +24v_IN; removed none
- sheet Can Transciever ports: added +3.3v_LSOM, SteeringCAN_H, SteeringCAN_L; removed CarCAN_H, CarCAN_L
Changed lines of the file:
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@@
 	(paper "A4")
 	(rectangle
-		(start 109.982 88.9)
+		(start 106.426 88.9)
 		(end 194.31 130.048)
 		(stroke
@@
 	(text "Steering Angle Sensor Components"
 		(exclude_from_sim no)
-		(at 135.128 86.614 0)
+		(at 131.318 86.868 0)
 		(effects
 			(font
@@
 	(wire
 		(pts
+			(xy 124.46 98.806) (xy 121.412 98.806)
+		)
+		(stroke
+			(width 0)
+			(type default)
+		)
+	)
+	(wire
+		(pts
 			(xy 176.022 103.886) (xy 176.53 103.378)
 		)
@@
 	(wire
 		(pts
+			(xy 121.412 98.806) (xy 119.38 96.774)
+		)
+		(stroke
+			(width 0)
+			(type default)
+		)
+	)
+	(wire
+		(pts
 			(xy 174.752 106.426) (xy 176.53 106.426)
 		)
@@
 	(wire
 		(pts
+			(xy 121.158 113.792) (xy 122.174 113.792)
+		)
+		(stroke
+			(width 0)
+			(type default)
+		)
+	)
+	(wire
+		(pts
+			(xy 120.142 119.634) (xy 122.174 119.634)
+		)
+		(stroke
+			(width 0)
+			(type default)
+		)
+	)
+	(wire
+		(pts
 			(xy 176.53 112.776) (xy 176.53 112.014)
 		)
@@
 	(wire
 		(pts
-			(xy 145.796 120.904) (xy 149.606 120.904)
-		)
-		(stroke
-			(width 0)
-			(type default)
-		)
-	)
-	(wire
-		(pts
-			(xy 145.796 117.094) (xy 149.606 117.094)
+			(xy 145.796 121.92) (xy 149.606 121.92)
+		)
+		(stroke
+			(width 0)
+			(type default)
+		)
+	)
+	(wire
+		(pts
+			(xy 145.796 117.094) (xy 149.86 117.094)
 		)
 		(stroke
@@
 	(wire
 		(pts
-			(xy 145.796 113.792) (xy 150.114 113.792)
-		)
-		(stroke
-			(width 0)
-			(type default)
-		)
-	)
-	(wire
-		(pts
-			(xy 121.92 113.792) (xy 124.46 113.792)
-		)
-		(stroke
-			(width 0)
-			(type default)
-		)
-	)
-	(wire
-		(pts
 			(xy 176.53 102.616) (xy 176.53 103.378)
 		)
@@
 	(wire
 		(pts
+			(xy 145.796 113.792) (xy 149.606 113.792)
+		)
+		(stroke
+			(width 0)
+			(type default)
+		)
+	)
+	(wire
+		(pts
 			(xy 146.05 98.806) (xy 148.59 98.806)
 		)
@@
 		)
 	)
-	(label "FDCAN1_RX"
+	(label "SteeringCAN_L"
+		(at 149.606 121.92 0)
+		(effects
+			(font
+				(size 1.27 1.27)
+			)
+			(justify left bottom)
+		)
+	)
+	(label "SteeringCAN_L"
 		(at 176.53 108.966 0)
 		(effects
@@
 		)
 	)
-	(label "FDCAN1_TX"
+	(label "SteeringCAN_H"
+		(at 149.86 117.094 0)
+		(effects
+			(font
+				(size 1.27 1.27)
+			)
+			(justify left bottom)
+		)
+	)
+	(label "SteeringCAN_H"
 		(at 176.53 106.426 0)
 		(effects
@@
 		)
 	)
-	(label "FDCAN1_TX"
-		(at 150.114 113.792 0)
+	(hierarchical_label "CAN_TX"
+		(shape input)
+		(at 149.606 113.792 0)
 		(effects
 			(font
 				(size 1.27 1.27)
 			)
-			(justify left bottom)
-		)
-	)
-	(label "FDCAN1_RX"
-		(at 121.92 113.792 180)
+			(justify left)
+		)
+	)
+	(hierarchical_label "CAN_RX"
+		(shape output)
+		(at 121.158 113.792 180)
 		(effects
 			(font
 				(size 1.27 1.27)
 			)
-			(justify right bottom)
-		)
-	)
-	(hierarchical_label "CarCAN_H"
+			(justify right)
+		)
+	)
+	(hierarchical_label "+3.3v_LSOM"
 		(shape input)
-		(at 149.606 117.094 0)
+		(at 120.142 119.634 180)
 		(effects
 			(font
 				(size 1.27 1.27)
 			)
-			(justify left)
-		)
-	)
-	(hierarchical_label "CarCAN_L"
-		(shape input)
-		(at 149.606 120.904 0)
-		(effects
-			(font
-				(size 1.27 1.27)
-			)
-			(justify left)
+			(justify right)
 		)
 	)
@@
 		)
 		(property "Value" "SteeringAngleConn_01x04"
-			(at 175.514 117.602 0)
+			(at 173.736 97.282 0)
 			(effects
 				(font
@@
 	(symbol
 		(lib_id "power:+24V")
+		(at 119.38 96.774 0)
+		(unit 1)
+		(exclude_from_sim no)
+		(in_bom yes)
+		(on_board yes)
+		(dnp no)
+		(property "Reference" "#PWR052"
+			(at 119.38 100.584 0)
+			(effects
+				(font
+					(size 1.27 1.27)
+				)
+				(hide yes)
+			)
+		)
+		(property "Value" "+24V"
+			(at 116.84 93.726 0)
+			(effects
+				(font
+					(size 1.27 1.27)
+				)
+			)
+		)
+		(property "Footprint" ""
+			(at 119.38 96.774 0)
+			(effects
+				(font
+					(size 1.27 1.27)
+				)
+				(hide yes)
+			)
+		)
+		(property "Datasheet" ""
+			(at 119.38 96.774 0)
+			(effects
+				(font
+					(size 1.27 1.27)
+				)
+				(hide yes)
+			)
+		)
+		(property "Description" "Power symbol creates a global label with name \"+24V\""
+			(at 119.38 96.774 0)
+			(effects
+				(font
+					(size 1.27 1.27)
+				)
+				(hide yes)
+			)
+		)
+		(pin "1"
+		)
+		(instances
+			(project "ControlsLeader_PCB"
+				(path "/298dad81-302c-41c7-874b-fcde1c3cde17/6f9c0058-7b30-4c81-afa5-092cb85861ec"
+					(reference "#PWR052")
+					(unit 1)
+				)
+			)
+		)
+	)
+	(symbol
+		(lib_id "power:+24V")
 		(at 176.53 102.616 0)
 		(unit 1)
@@
 	)
 	(sheet
-		(at 124.46 110.998)
-		(size 21.336 12.954)
+		(at 122.174 110.998)
+		(size 23.622 12.954)
 		(exclude_from_sim no)
 		(in_bom yes)
@@
 		)
 		(property "Sheetname" "Can Transciever"
-			(at 127.254 110.236 0)
+			(at 124.968 110.236 0)
 			(effects
 				(font
@@
 		)
 		(property "Sheetfile" "CanTransciever.kicad_sch"
-			(at 121.666 125.222 0)
+			(at 119.38 125.222 0)
 			(effects
 				(font
@@
 		)
 		(pin "CAN_RX" output
-			(at 124.46 113.792 180)
+			(at 122.174 113.792 180)
 			(effects
 				(font
@@
 			)
 		)
-		(pin "CarCAN_H" input
+		(pin "SteeringCAN_H" input
 			(at 145.796 117.094 0)
 			(effects
@@
 			)
 		)
-		(pin "CarCAN_L" input
-			(at 145.796 120.904 0)
+		(pin "SteeringCAN_L" input
+			(at 145.796 121.92 0)
 			(effects
 				(font
@@
 				)
 				(justify right)
+			)
+		)
+		(pin "+3.3v_LSOM" input
+			(at 122.174 119.634 180)
+			(effects
+				(font
+					(size 1.27 1.27)
+				)
+				(justify left)
 			)
 		)
@@
 			)
 		)
+		(pin "+24v_IN" input
+			(at 124.46 98.806 180)
+			(effects
+				(font
+					(size 1.27 1.27)
+				)
+				(justify left)
+			)
+		)
