File: hardware/ControlsLeader_PCB/Steering_Wheel.kicad_sch (KiCad schematic)
At the start: 6 parts, among them J10 Indicator_Switch, Q6 NMOS

Commit message: ShaqDash is born. . . RPP in progress
Parts:
- removed F2: Fuse, Fuse:Fuseholder_Blade_Mini_Keystone_3568, symbol Device:Fuse
Connections:
- net Horn_24V_Signal_Out: now also Q6.1 (D)
- net 3.3V_LDO renamed 5V_Buck
- net Horn_3.3V_Signal renamed Horn_5V_Signal
Other:
- sheet NMOS Switch1 ports: added 5V_Switch_Signal; removed 3.3V_Switch_Signal
- sheet NMOS Switch2 ports: added 5V_Switch_Signal; removed 3.3V_Switch_Signal
- sheet NMOS Switch3 ports: added 5V_Switch_Signal; removed 3.3V_Switch_Signal
- sheet NMOS Switch8 ports: added 5V_Switch_Signal; removed 3.3V_Switch_Signal
- moved on the sheet: Horn2, J10, Regen_Active1

Commit message: revb layout, working on silkscreen
Parts:
- removed Q6: NMOS, LSOM_IRLM:SOT23, symbol Simulation_SPICE:NMOS
- added Q6: NVMFWS1D7N04XMT1G, NVMFWS3D0P04M8LT1G:NVMFWS3D0P04M8LT1G, symbol NVMFWS1D7N04XMT1G:NVMFWS1D7N04XMT1G
Connections:
- net GND: now also Q6.1, Q6.2, Q6.3
- net Horn_24V_Signal_Out: now also Q6.5, Q6.6, Q6.7, Q6.8, Q6.9
- net Horn_GPIO_OUT: now also Q6.4
Other:
- added sheet NMOS Switch9 (NMOS_SW.kicad_sch)
- note added: "Push to Talk >:("
- moved on the sheet: Horn2, J10, Regen_Active1
