File: hardware/ControlsLeader_PCB/steeringAngleLDO.kicad_sch (KiCad schematic)
At the start: 12 parts, among them IC2 AP2205-W5-7

Commit message: revb layout, working on silkscreen
Parts:
- renumbered 5V_Out1 to 16v_Out1, Adj5V1 to Adj16V1, En5V1 to En16V1
Connections:
- net 16v_prefuse: now reaches 16v_Out1.1, C27.1, F1.1, IC2.5 (VOUT), R65.1
- net +24V renamed +24v_IN
Other:
- moved on the sheet: 16v_Out1
Changed lines of the file:
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@@
+	)
+	(junction
+		(at 144.526 94.742)
+		(diameter 0)
+		(color 0 0 0 0)
 	)
 	(junction
@@
 	)
 	(junction
-		(at 152.654 94.742)
-		(diameter 0)
-		(color 0 0 0 0)
-	)
-	(junction
 		(at 104.648 92.202)
 		(diameter 0)
@@
 	)
 	(junction
+		(at 157.734 94.742)
+		(diameter 0)
+		(color 0 0 0 0)
+	)
+	(junction
 		(at 114.046 92.202)
 		(diameter 0)
@@
 	(wire
 		(pts
+			(xy 144.526 94.742) (xy 147.32 94.742)
+		)
+		(stroke
+			(width 0)
+			(type default)
+		)
+	)
+	(wire
+		(pts
 			(xy 155.956 94.742) (xy 155.956 98.806)
 		)
@@
 	(wire
 		(pts
-			(xy 147.32 94.742) (xy 152.654 94.742)
+			(xy 144.526 92.71) (xy 144.526 94.742)
+		)
+		(stroke
+			(width 0)
+			(type default)
+		)
+	)
+	(wire
+		(pts
+			(xy 147.32 94.742) (xy 155.956 94.742)
 		)
 		(stroke
@@
 	(wire
 		(pts
+			(xy 157.734 94.742) (xy 157.988 94.742)
+		)
+		(stroke
+			(width 0)
+			(type default)
+		)
+	)
+	(wire
+		(pts
 			(xy 107.442 108.966) (xy 107.442 109.728)
 		)
@@
 	(wire
 		(pts
-			(xy 155.956 94.742) (xy 157.988 94.742)
-		)
-		(stroke
-			(width 0)
-			(type default)
-		)
-	)
-	(wire
-		(pts
-			(xy 152.654 94.742) (xy 155.956 94.742)
+			(xy 155.956 94.742) (xy 157.734 94.742)
 		)
 		(stroke
@@
 	(wire
 		(pts
-			(xy 144.018 94.742) (xy 147.32 94.742)
+			(xy 144.018 94.742) (xy 144.526 94.742)
 		)
 		(stroke
@@
 	(wire
 		(pts
+			(xy 103.632 89.662) (xy 103.632 91.186)
+		)
+		(stroke
+			(width 0)
+			(type default)
+		)
+	)
+	(wire
+		(pts
 			(xy 155.448 110.998) (xy 155.956 110.49)
 		)
@@
 	(wire
 		(pts
-			(xy 103.632 90.932) (xy 103.632 91.186)
-		)
-		(stroke
-			(width 0)
-			(type default)
-		)
-	)
-	(wire
-		(pts
 			(xy 152.146 110.998) (xy 155.448 110.998)
 		)
@@
 			(width 0)
 			(type default)
+		)
+	)
+	(label "16v_prefuse"
+		(at 144.526 92.71 0)
+		(effects
+			(font
+				(size 1.27 1.27)
+			)
+			(justify left bottom)
 		)
 	)
@@
 			)
 			(justify left)
+		)
+	)
+	(hierarchical_label "+24v_IN"
+		(shape input)
+		(at 103.632 89.662 180)
+		(effects
+			(font
+				(size 1.27 1.27)
+			)
+			(justify right)
 		)
 	)
@@
 		(dnp no)
 		(property "Reference" "C26"
-			(at 113.284 106.68 0)
+			(at 114.554 106.68 0)
 			(effects
 				(font
@@
 		(on_board yes)
 		(dnp no)
-		(property "Reference" "Adj5V1"
+		(property "Reference" "Adj16V1"
 			(at 144.272 104.648 90)
 			(effects
@@
 			(project "ControlsLeader_PCB"
 				(path "/298dad81-302c-41c7-874b-fcde1c3cde17/6f9c0058-7b30-4c81-afa5-092cb85861ec/d2a39224-ea42-493b-ad1b-fc800fa3b4ea"
-					(reference "Adj5V1")
+					(reference "Adj16V1")
 					(unit 1)
 				)
@@
 	(symbol
 		(lib_id "Connector:TestPoint")
-		(at 152.654 94.742 0)
+		(at 157.734 94.742 0)
 		(unit 1)
 		(exclude_from_sim no)
@@
 		(on_board yes)
 		(dnp no)
-		(property "Reference" "5V_Out1"
-			(at 156.21 88.646 0)
+		(property "Reference" "16v_Out1"
+			(at 161.29 88.646 0)
 			(effects
 				(font
@@
 		)
 		(property "Value" "5V_Out"
-			(at 155.448 89.154 0)
+			(at 160.528 89.154 0)
 			(effects
 				(font
@@
 		)
 		(property "Footprint" "TestPoint:TestPoint_Pad_1.0x1.0mm"
+			(at 162.814 94.742 0)
+			(effects
+				(font
+					(size 1.27 1.27)
+				)
+				(hide yes)
+			)
+		)
+		(property "Datasheet" "~"
+			(at 162.814 94.742 0)
+			(effects
+				(font
+					(size 1.27 1.27)
+				)
+				(hide yes)
+			)
+		)
+		(property "Description" "test point"
 			(at 157.734 94.742 0)
 			(effects
@@
 			)
 		)
-		(property "Datasheet" "~"
+		(property "P/N" "~"
 			(at 157.734 94.742 0)
 			(effects
@@
 			)
 		)
-		(property "Description" "test point"
-			(at 152.654 94.742 0)
-			(effects
-				(font
-					(size 1.27 1.27)
-				)
-				(hide yes)
-			)
-		)
-		(property "P/N" "~"
-			(at 152.654 94.742 0)
-			(effects
-				(font
-					(size 1.27 1.27)
-				)
-				(hide yes)
-			)
-		)
 		(property "Silkscreen" ""
-			(at 152.654 94.742 0)
+			(at 157.734 94.742 0)
 			(effects
 				(font
@@
 		)
 		(property "Sim.Library" ""
-			(at 152.654 94.742 0)
+			(at 157.734 94.742 0)
 			(effects
 				(font
@@
 		)
 		(property "Sim.Name" ""
-			(at 152.654 94.742 0)
+			(at 157.734 94.742 0)
 			(effects
 				(font
@@
 			(project "ControlsLeader_PCB"
 				(path "/298dad81-302c-41c7-874b-fcde1c3cde17/6f9c0058-7b30-4c81-afa5-092cb85861ec/d2a39224-ea42-493b-ad1b-fc800fa3b4ea"
-					(reference "5V_Out1")
+					(reference "16v_Out1")
 					(unit 1)
 				)
@@
 		(on_board yes)
 		(dnp no)
-		(property "Reference" "En5V1"
+		(property "Reference" "En16V1"
 			(at 117.602 101.854 90)
 			(effects
@@
 			(project "ControlsLeader_PCB"
 				(path "/298dad81-302c-41c7-874b-fcde1c3cde17/6f9c0058-7b30-4c81-afa5-092cb85861ec/d2a39224-ea42-493b-ad1b-fc800fa3b4ea"
-					(reference "En5V1")
-					(unit 1)
-				)
-			)
-		)
-	)
-	(symbol
-		(lib_id "power:+24V")
-		(at 103.632 90.932 0)
-		(unit 1)
-		(exclude_from_sim no)
-		(in_bom yes)
-		(on_board yes)
-		(dnp no)
-		(property "Reference" "#PWR052"
-			(at 103.632 94.742 0)
-			(effects
-				(font
-					(size 1.27 1.27)
-				)
-				(hide yes)
-			)
-		)
-		(property "Value" "+24V"
-			(at 101.092 87.884 0)
-			(effects
-				(font
-					(size 1.27 1.27)
-				)
-			)
-		)
-		(property "Footprint" ""
-			(at 103.632 90.932 0)
-			(effects
-				(font
-					(size 1.27 1.27)
-				)
-				(hide yes)
-			)
-		)
-		(property "Datasheet" ""
-			(at 103.632 90.932 0)
-			(effects
-				(font
-					(size 1.27 1.27)
-				)
-				(hide yes)
-			)
-		)
-		(property "Description" "Power symbol creates a global label with name \"+24V\""
-			(at 103.632 90.932 0)
-			(effects
-				(font
-					(size 1.27 1.27)
-				)
-				(hide yes)
-			)
-		)
-		(pin "1"
-		)
-		(instances
-			(project "ControlsLeader_PCB"
-				(path "/298dad81-302c-41c7-874b-fcde1c3cde17/6f9c0058-7b30-4c81-afa5-092cb85861ec/d2a39224-ea42-493b-ad1b-fc800fa3b4ea"
-					(reference "#PWR052")
+					(reference "En16V1")
 					(unit 1)
 				)
@@
 		(dnp no)
 		(property "Reference" "R65"
-			(at 149.098 99.06 0)
+			(at 148.59 99.06 0)
 			(effects
 				(font
@@
 		(dnp no)
 		(property "Reference" "R66"
-			(at 149.606 106.68 0)
-			(effects
-				(font
+			(at 148.59 106.68 0)
+			(effects
+				(font
