File: hardware/ControlsLeader_PCB/CanTransciever.kicad_sch (KiCad schematic)
At the start: 7 parts, among them IC1 TCAN337DCNR, U1 CDSOT23-T24CAN

Commit message: revb layout, working on silkscreen
Parts:
- added CC_Term1: Jumper_2_Open, Connector_PinHeader_2.54mm:PinHeader_1x02_P2.54mm_Vertical, symbol Jumper:Jumper_2_Open
- added R68: 120, Resistor_SMD:R_0603_1608Metric_Pad0.98x0.95mm_HandSolder, symbol Device:R
Connections:
- net +3V3 renamed +3.3v_LSOM
- net CarCAN_H renamed SteeringCAN_H
- net SteeringCAN_H: now also R68.2
- net CarCAN_L renamed SteeringCAN_L
- net SteeringCAN_L: now also CC_Term1.2 (B)
- new net: CC_Term1.1 (A), R68.1
Other:
- note added: "CAN Bus Termination"

Commit message: Final fixes
Parts:
- added CC_Term2: Jumper_2_Open, Connector_PinHeader_2.54mm:PinHeader_1x02_P2.54mm_Vertical, symbol Jumper:Jumper_2_Open
Connections:
- net CAN_RX: now also CC_Term2.1 (A)
- net CAN_TX: now also CC_Term2.2 (B)
Changed lines of the file:
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@@
 	(paper "A4")
 	(rectangle
-		(start 72.39 73.66)
+		(start 65.024 73.66)
 		(end 212.217 119.38)
 		(stroke
@@
 	(wire
 		(pts
+			(xy 84.836 106.172) (xy 85.09 106.172)
+		)
+		(stroke
+			(width 0)
+			(type default)
+		)
+	)
+	(wire
+		(pts
 			(xy 84.582 85.344) (xy 85.598 84.328)
 		)
@@
 	(wire
 		(pts
+			(xy 85.09 111.252) (xy 88.138 114.3)
+		)
+		(stroke
+			(width 0)
+			(type default)
+		)
+	)
+	(wire
+		(pts
+			(xy 89.408 114.3) (xy 89.662 114.046)
+		)
+		(stroke
+			(width 0)
+			(type default)
+		)
+	)
+	(wire
+		(pts
 			(xy 125.984 90.17) (xy 141.224 90.17)
 		)
@@
 	(wire
 		(pts
+			(xy 85.09 106.172) (xy 87.884 103.378)
+		)
+		(stroke
+			(width 0)
+			(type default)
+		)
+	)
+	(wire
+		(pts
 			(xy 141.224 103.632) (xy 143.764 103.632)
 		)
@@
 	(wire
 		(pts
+			(xy 87.884 103.378) (xy 89.154 103.378)
+		)
+		(stroke
+			(width 0)
+			(type default)
+		)
+	)
+	(wire
+		(pts
 			(xy 113.284 81.026) (xy 113.284 82.55)
 		)
@@
 	(wire
 		(pts
+			(xy 89.154 103.378) (xy 89.662 103.886)
+		)
+		(stroke
+			(width 0)
+			(type default)
+		)
+	)
+	(wire
+		(pts
 			(xy 137.922 95.25) (xy 146.812 95.25)
 		)
@@
 		(pts
 			(xy 143.764 106.172) (xy 137.922 106.172)
+		)
+		(stroke
+			(width 0)
+			(type default)
+		)
+	)
+	(wire
+		(pts
+			(xy 88.138 114.3) (xy 89.408 114.3)
 		)
 		(stroke
@@
 		)
 	)
+	(hierarchical_label "CAN_TX"
+		(shape input)
+		(at 84.836 106.172 180)
+		(effects
+			(font
+				(size 1.27 1.27)
+			)
+			(justify right)
+		)
+	)
 	(hierarchical_label "+3.3v_LSOM"
 		(shape input)
@@
 			)
 			(justify left)
+		)
+	)
+	(hierarchical_label "CAN_RX"
+		(shape output)
+		(at 85.09 111.252 180)
+		(effects
+			(font
+				(size 1.27 1.27)
+			)
+			(justify right)
 		)
 	)
@@
 					(unit 1)
 				)
+			)
+		)
+	)
+	(symbol
+		(lib_id "Jumper:Jumper_2_Open")
+		(at 89.662 108.966 90)
+		(unit 1)
+		(exclude_from_sim no)
+		(in_bom no)
+		(on_board yes)
+		(dnp no)
+		(property "Reference" "CC_Term2"
+			(at 91.694 109.093 0)
+			(effects
+				(font
+					(size 1.27 1.27)
+				)
+			)
+		)
+		(property "Value" "Jumper_2_Open"
+			(at 94.234 109.093 0)
+			(effects
+				(font
+					(size 1.27 1.27)
+				)
+			)
+		)
+		(property "Footprint" "Connector_PinHeader_2.54mm:PinHeader_1x02_P2.54mm_Vertical"
+			(at 89.662 108.966 0)
+			(effects
+				(font
+					(size 1.27 1.27)
+				)
+				(hide yes)
+			)
+		)
+		(property "Datasheet" "~"
+			(at 89.662 108.966 0)
+			(effects
+				(font
+					(size 1.27 1.27)
+				)
+				(hide yes)
+			)
+		)
+		(property "Description" "Jumper, 2-pole, open"
+			(at 89.662 108.966 0)
+			(effects
+				(font
+					(size 1.27 1.27)
+				)
+				(hide yes)
+			)
+		)
+		(property "PN" ""
+			(at 89.662 108.966 0)
+			(effects
+				(font
+					(size 1.27 1.27)
+				)
+				(hide yes)
+			)
+		)
+		(property "p/n" ""
+			(at 89.662 108.966 0)
+			(effects
+				(font
+					(size 1.27 1.27)
+				)
+				(hide yes)
+			)
+		)
+		(property "Color" ""
+			(at 89.662 108.966 0)
+			(effects
+				(font
+					(size 1.27 1.27)
+				)
+			)
+		)
+		(property "If" ""
+			(at 89.662 108.966 0)
+			(effects
+				(font
+					(size 1.27 1.27)
+				)
+			)
+		)
+		(property "Mfg" ""
+			(at 89.662 108.966 0)
+			(effects
+				(font
+					(size 1.27 1.27)
+				)
+			)
+		)
+		(property "Vf" ""
+			(at 89.662 108.966 0)
+			(effects
+				(font
+					(size 1.27 1.27)
+				)
+			)
+		)
+		(pin "2"
+		)
+		(pin "1"
+		)
+		(instances
+			(project "ControlsLeader_PCB"
+				(path "/298dad81-302c-41c7-874b-fcde1c3cde17/6f9c0058-7b30-4c81-afa5-092cb85861ec/b0729058-c6be-49c1-a87e-2ac8a37e6931"
+					(reference "CC_Term2")
+					(unit 1)
+				)
