File: hardware/ControlsLeader_PCB/ControlsLeader_PCB.kicad_sch (KiCad schematic)
At the start: 20 parts, among them J1 CarCANConnector_Out, J12 SteeringConn_01x07, J15 IgnConn_01x04, J17 Conn_01x02, J2 PeripheralCAN_out, J3 CarCANConnector_In, J4 PeripheralCAN_in, J6 Conn_2Rows-13Pins, J8 Dash_Lsom_Horn_Lights_PWR, U2 LeaderSOM

Commit message: ShaqDash is born. . . RPP in progress
Parts:
- removed D30: Controls_Leader_Status_Red, LED_SMD:LED_0603_1608Metric_Pad1.05x0.95mm_HandSolder, symbol Device:LED
- removed F1: Fuse, Fuse:Fuseholder_Blade_Mini_Keystone_3568, symbol Device:Fuse
- removed J12: SteeringConn_01x07, Connector_Molex:Molex_Nano-Fit_105313-xx07_1x07_P2.50mm_Horizontal, symbol Connector_Generic:Conn_01x07
- removed R56: 1.1k, Resistor_SMD:R_0603_1608Metric_Pad0.98x0.95mm_HandSolder, symbol Device:R
- added F2, F3: Fuse, Fuse:Fuseholder_Blade_Mini_Keystone_3568, symbol Device:Fuse
- added J14: SteeringConn_01x06, Connector_Molex:Molex_Nano-Fit_105313-xx06_1x06_P2.50mm_Horizontal, symbol Connector_Generic:Conn_01x06
- D29: footprint Diode_SMD:D_SOD-523 -> Diode_SMD:D_SOD-123F
Connections:
- net 3.3V_LDO is gone; now on net 5V_LDO: J15.1 (Pin_1), J6.1 (Pin_1), J6.3 (Pin_3), J6.5 (Pin_5), J6.7 (Pin_7), J6.9 (Pin_9)
- net +24V: no longer J8.1 (Pin_1)
- net +24v_Horn: now also F2.1; no longer J8.3 (Pin_3)
- net +24v_Lights: now also F3.2; no longer J8.2 (Pin_2)
- net 5V_LDO: now also J14.6 (Pin_6)
- net Indicator_PWM: now also J14.5 (Pin_5)
- net Left_Blinker_Signal: now also J14.1 (Pin_1)
- net Regen_Active_Signal: now also J14.4 (Pin_4)
- net Right_Blinker_Signal: now also J14.2 (Pin_2)
- new net: F3.1, J8.2 (Pin_2)
- new net: F2.2, J8.3 (Pin_3)
- new net Horn_5V_Signal: J14.3 (Pin_3)
- new net RPP/24v_Ext: J8.1 (Pin_1)
Other:
- removed sheet 5v_3.3v_LDO
- added sheet RPP (RPP.kicad_sch)
- sheet Dash ports: added 5V_Buck; removed 3.3V_LDO
- sheet Steering_Wheel ports: added 5V_Buck, Horn_5V_Signal; removed 3.3V_LDO, Horn_3.3V_Signal
- moved on the sheet: D28, D29, J17, J8, R10, U2A, U2B

Commit message: Steering Angle Sensor SCH changes
Parts:
- added R60, R61: 0, Resistor_SMD:R_0603_1608Metric_Pad0.98x0.95mm_HandSolder, symbol Device:R
Connections:
- net +24V: now also R60.2, R61.2
- net at F3.1, J8.2 (Pin_2): now also R61.1
- net at F2.2, J8.3 (Pin_3): now also R60.1
- net 5V_LDO renamed 5V_Buck
Other:
- added sheet Steering Angle Sensor Components (SteerinAngle.kicad_sch)
- moved on the sheet: D28, D29, F2, F3, J14, J17, R10

Commit message: revb layout, working on silkscreen
Parts:
- added F4, F5: 0603L025YR, 0603L025YR:FUSC1608X75N, symbol 0603L025YR:0603L025YR
- added J16: Conn_01x03, Connector_Molex:Molex_Nano-Fit_105313-xx03_1x03_P2.50mm_Horizontal, symbol Connector_Generic:Conn_01x03
Connections:
- net 5V_Buck: now also F4.1, F5.1; no longer J14.6 (Pin_6), J6.1 (Pin_1), J6.3 (Pin_3), J6.5 (Pin_5), J6.7 (Pin_7), J6.9 (Pin_9)
- net GND: now also J16.1 (Pin_1)
- net Indicator_PWM: now also J16.2 (Pin_2); no longer J14.5 (Pin_5)
- net Extra_LED1 renamed FDCAN2_TX
- net Extra_LED3 renamed FDCAN2_RX
- net Extra_LED4 renamed PTT_GPIO_IN
- new net 5V_Buck_IndicationLights: F4.2, J16.3 (Pin_3)
- new net 5V_Buck_SteeringDash: F5.2, J14.6 (Pin_6), J6.1 (Pin_1), J6.3 (Pin_3), J6.5 (Pin_5), J6.7 (Pin_7), J6.9 (Pin_9)
- new net PTT_Signal: J14.5 (Pin_5)
Other:
- sheet Status_LEDs ports: added none; removed Extra_LED1, Extra_LED3, Extra_LED4
- sheet Steering Angle Sensor Components ports: added +3.3v_LSOM, CAN_RX, CAN_TX; removed CarCAN_H, CarCAN_L
- sheet Steering_Wheel ports: added PTT_GPIO_IN, PTT_Signal; removed none
- note added: "Dash Lights"
- moved on the sheet: J14

Commit message: Final fixes
Parts:
- removed F4: 0603L025YR, 0603L025YR:FUSC1608X75N, symbol 0603L025YR:0603L025YR
- added F4: 0805L100WR, FUSC2114X180N, symbol 0805L100WR:0805L100WR
Connections:
- net 5V_Buck: now also F4.1
- net 5V_Buck_IndicationLights: now also F4.2
Changed lines of the file:
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@@
 	(wire
 		(pts
-			(xy 248.666 177.038) (xy 250.19 177.038)
+			(xy 248.666 178.054) (xy 250.19 178.054)
 		)
 		(stroke
@@
 	(wire
 		(pts
-			(xy 267.97 177.038) (xy 268.732 177.038)
+			(xy 267.97 178.054) (xy 268.732 178.054)
 		)
 		(stroke
@@
 	)
 	(label "5V_Buck"
-		(at 248.666 177.038 180)
+		(at 248.666 178.054 180)
 		(effects
 			(font
@@
 	)
 	(label "5V_Buck_IndicationLights"
-		(at 268.732 177.038 0)
+		(at 268.732 178.054 0)
 		(effects
 			(font
@@
 	)
 	(symbol
+		(lib_id "0805L100WR:0805L100WR")
+		(at 250.19 178.054 0)
+		(unit 1)
+		(exclude_from_sim no)
+		(in_bom yes)
+		(on_board yes)
+		(dnp no)
+		(property "Reference" "F4"
+			(at 259.334 175.514 0)
+			(effects
+				(font
+					(size 1.27 1.27)
+				)
+			)
+		)
+		(property "Value" "0805L100WR"
+			(at 250.952 175.514 0)
+			(effects
+				(font
+					(size 1.27 1.27)
+				)
+			)
+		)
+		(property "Footprint" "FUSC2114X180N"
+			(at 264.16 274.244 0)
+			(effects
+				(font
+					(size 1.27 1.27)
+				)
+				(justify left top)
+				(hide yes)
+			)
+		)
+		(property "Datasheet" "https://www.arrow.com/en/products/0805l100wr/littelfuse"
+			(at 264.16 374.244 0)
+			(effects
+				(font
+					(size 1.27 1.27)
+				)
+				(justify left top)
+				(hide yes)
+			)
+		)
+		(property "Description" "LITTELFUSE - 0805L100WR - Resettable Fuse, PPTC, 0805 (2012 Metric), POLYFUSE 0805L, 6 VDC, 1 A, 1.95 A, 0.3 s"
+			(at 250.19 178.054 0)
+			(effects
+				(font
+					(size 1.27 1.27)
+				)
+				(hide yes)
+			)
+		)
+		(property "Height" "1.8"
+			(at 264.16 574.244 0)
+			(effects
+				(font
+					(size 1.27 1.27)
+				)
+				(justify left top)
+				(hide yes)
+			)
+		)
+		(property "Mouser Part Number" "576-0805L100"
+			(at 264.16 674.244 0)
+			(effects
+				(font
+					(size 1.27 1.27)
+				)
+				(justify left top)
+				(hide yes)
+			)
+		)
+		(property "Mouser Price/Stock" "https://www.mouser.co.uk/ProductDetail/Littelfuse/0805L100WR?qs=SJZ%252BTX%252BI2BTMlREVsW49pQ%3D%3D"
+			(at 264.16 774.244 0)
+			(effects
+				(font
+					(size 1.27 1.27)
+				)
+				(justify left top)
+				(hide yes)
+			)
+		)
+		(property "Manufacturer_Name" "LITTELFUSE"
+			(at 264.16 874.244 0)
+			(effects
+				(font
+					(size 1.27 1.27)
+				)
+				(justify left top)
+				(hide yes)
+			)
+		)
+		(property "Manufacturer_Part_Number" "0805L100WR"
+			(at 264.16 974.244 0)
+			(effects
+				(font
+					(size 1.27 1.27)
+				)
+				(justify left top)
+				(hide yes)
+			)
+		)
+		(pin "2"
+		)
+		(pin "1"
+		)
+		(instances
+			(project ""
+				(path "/298dad81-302c-41c7-874b-fcde1c3cde17"
+					(reference "F4")
+					(unit 1)
+				)
+			)
+		)
+	)
+	(symbol
 		(lib_id "Mechanical:MountingHole")
 		(at 25.4 191.77 0)
@@
 		(dnp no)
 		(property "Reference" "F5"
-			(at 259.334 179.832 0)
+			(at 259.08 168.656 0)
 			(effects
 				(font
@@
 		)
 		(property "Value" "0603L025YR"
-			(at 251.206 179.578 0)
+			(at 251.206 168.656 0)
 			(effects
 				(font
@@
 					(unit 1)
 				)
-			)
-		)
-	)
-	(symbol
-		(lib_id "0603L025YR:0603L025YR")
-		(at 250.19 177.038 0)
-		(unit 1)
-		(exclude_from_sim no)
-		(in_bom yes)
-		(on_board yes)
-		(dnp no)
-		(property "Reference" "F4"
-			(at 258.826 173.99 0)
-			(effects
-				(font
-					(size 1.27 1.27)
-				)
-			)
-		)
-		(property "Value" "0603L025YR"
-			(at 251.46 173.736 0)
-			(effects
-				(font
-					(size 1.27 1.27)
-				)
-			)
-		)
-		(property "Footprint" "0603L025YR:FUSC1608X75N"
-			(at 264.16 273.228 0)
-			(effects
-				(font
-					(size 1.27 1.27)
-				)
-				(justify left top)
-				(hide yes)
-			)
-		)
-		(property "Datasheet" "https://m.littelfuse.com/~/media/electronics/datasheets/resettable_ptcs/littelfuse_ptc_0603l_datasheet.pdf.pdf"
-			(at 264.16 373.228 0)
-			(effects
-				(font
-					(size 1.27 1.27)
-				)
-				(justify left top)
-				(hide yes)
-			)
-		)
-		(property "Description" "Resettable Fuses - PPTC PTC 9V .250A POLY SURF MOUNT"
-			(at 250.19 177.038 0)
-			(effects
-				(font
-					(size 1.27 1.27)
-				)
-				(hide yes)
-			)
-		)
-		(property "Height" "0.75"
-			(at 264.16 573.228 0)
-			(effects
-				(font
-					(size 1.27 1.27)
-				)
-				(justify left top)
-				(hide yes)
-			)
-		)
-		(property "Mouser Part Number" "576-0603L025YR"
-			(at 264.16 673.228 0)
-			(effects
-				(font
-					(size 1.27 1.27)
-				)
-				(justify left top)
-				(hide yes)
-			)
-		)
-		(property "Mouser Price/Stock" "https://www.mouser.co.uk/ProductDetail/Littelfuse/0603L025YR?qs=n5MbhIql%252BRmYmNliBUCDFQ%3D%3D"
-			(at 264.16 773.228 0)
-			(effects
-				(font
-					(size 1.27 1.27)
-				)
-				(justify left top)
-				(hide yes)
-			)
-		)
-		(property "Manufacturer_Name" "LITTELFUSE"
-			(at 264.16 873.228 0)
-			(effects
-				(font
-					(size 1.27 1.27)
-				)
-				(justify left top)
-				(hide yes)
-			)
-		)
-		(property "Manufacturer_Part_Number" "0603L025YR"
-			(at 264.16 973.228 0)
-			(effects
-				(font
-					(size 1.27 1.27)
-				)
-				(justify left top)
-				(hide yes)
-			)
-		)
-		(property "Silkscreen" ""
-			(at 250.19 177.038 0)
-			(effects
-				(font
-					(size 1.27 1.27)
-				)
-				(hide yes)
-			)
-		)
-		(property "Sim.Library" ""
-			(at 250.19 177.038 0)
-			(effects
-				(font
-					(size 1.27 1.27)
-				)
-				(hide yes)
-			)
-		)
-		(property "Sim.Name" ""
-			(at 250.19 177.038 0)
-			(effects
-				(font
-					(size 1.27 1.27)
-				)
-				(hide yes)
-			)
-		)
-		(pin "2"
-		)
-		(pin "1"
-		)
-		(instances
-			(project "ControlsLeader_PCB"
-				(path "/298dad81-302c-41c7-874b-fcde1c3cde17"
-					(reference "F4")
-					(unit 1)
-				)
