File: hardware/ControlsLeader_PCB/ControlsLeader_PCB.kicad_sch (KiCad schematic)
At the start: 20 parts, among them J1 CarCANConnector_Out, J12 SteeringConn_01x07, J15 IgnConn_01x04, J17 Conn_01x02, J2 PeripheralCAN_out, J3 CarCANConnector_In, J4 PeripheralCAN_in, J6 Conn_2Rows-13Pins, J8 Dash_Lsom_Horn_Lights_PWR, U2 LeaderSOM

Commit message: Mika is quite smart (#12)
Parts:
- removed D30: Controls_Leader_Status_Red, LED_SMD:LED_0603_1608Metric_Pad1.05x0.95mm_HandSolder, symbol Device:LED
- removed F1: Fuse, Fuse:Fuseholder_Blade_Mini_Keystone_3568, symbol Device:Fuse
- removed J12: SteeringConn_01x07, Connector_Molex:Molex_Nano-Fit_105313-xx07_1x07_P2.50mm_Horizontal, symbol Connector_Generic:Conn_01x07
- removed R56: 1.1k, Resistor_SMD:R_0603_1608Metric_Pad0.98x0.95mm_HandSolder, symbol Device:R
- added F2, F3: Fuse, Fuse:Fuseholder_Blade_Mini_Keystone_3568, symbol Device:Fuse
- added F4: 0805L100WR, FUSC2114X180N, symbol 0805L100WR:0805L100WR
- added F5: 0603L025YR, 0603L025YR:FUSC1608X75N, symbol 0603L025YR:0603L025YR
- added J14: SteeringConn_01x06, Connector_Molex:Molex_Nano-Fit_105313-xx06_1x06_P2.50mm_Horizontal, symbol Connector_Generic:Conn_01x06
- added J16: Conn_01x03, Connector_Molex:Molex_Nano-Fit_105313-xx03_1x03_P2.50mm_Horizontal, symbol Connector_Generic:Conn_01x03
- added R60, R61: 0, Resistor_SMD:R_0603_1608Metric_Pad0.98x0.95mm_HandSolder, symbol Device:R
- D29: footprint Diode_SMD:D_SOD-523 -> Diode_SMD:D_SOD-123F
Connections:
- net +24V: now also R60.2, R61.2; no longer J8.1 (Pin_1)
- net +24v_Horn: now also F2.1; no longer J8.3 (Pin_3)
- net +24v_Lights: now also F3.2; no longer J8.2 (Pin_2)
- net GND: now also J16.1 (Pin_1)
- net Indicator_PWM: now also J16.2 (Pin_2)
- net Left_Blinker_Signal: now also J14.1 (Pin_1)
- net Regen_Active_Signal: now also J14.4 (Pin_4)
- net Right_Blinker_Signal: now also J14.2 (Pin_2)
- net 3.3V_LDO renamed 5V_Buck_SteeringDash
- net 5V_Buck_SteeringDash: now also F5.2, J14.6 (Pin_6); no longer J15.1 (Pin_1)
- net 5V_LDO renamed 5V_Buck
- net 5V_Buck: now also J15.1 (Pin_1), F4.1, F5.1
- net Extra_LED1 renamed FDCAN2_TX
- net Extra_LED3 renamed FDCAN2_RX
- net Extra_LED4 renamed PTT_GPIO_IN
- new net: F3.1, J8.2 (Pin_2), R61.1
- new net: F2.2, J8.3 (Pin_3), R60.1
- new net 5V_Buck_IndicationLights: F4.2, J16.3 (Pin_3)
- new net Horn_5V_Signal: J14.3 (Pin_3)
- new net PTT_Signal: J14.5 (Pin_5)
- new net RPP/24v_Ext: J8.1 (Pin_1)
Other:
- removed sheet 5v_3.3v_LDO
- added sheet RPP (RPP.kicad_sch)
- added sheet Steering Angle Sensor Components (SteerinAngle.kicad_sch)
- sheet Dash ports: added 5V_Buck; removed 3.3V_LDO
- sheet Status_LEDs ports: added none; removed Extra_LED1, Extra_LED3, Extra_LED4
- sheet Steering_Wheel ports: added 5V_Buck, Horn_5V_Signal, PTT_GPIO_IN, PTT_Signal; removed 3.3V_LDO, Horn_3.3V_Signal
- note added: "Dash Lights"
- moved on the sheet: D28, J8, R10, U2A, U2B
