File: hardware/ControlsLeader_PCB/dash.kicad_sch (KiCad schematic)
At the start: 10 parts, among them J11 EStop1, J13 Supp_Out, J7 Conn_01x04, J9 Supp_In

Commit message: Mika is quite smart (#12)
Connections:
- net 3.3V_LDO renamed 5V_Buck
Other:
- sheet NMOS Switch ports: added 5V_Switch_Signal; removed 3.3V_Switch_Signal
- sheet NMOS Switch1 ports: added 5V_Switch_Signal; removed 3.3V_Switch_Signal
- sheet NMOS Switch2 ports: added 5V_Switch_Signal; removed 3.3V_Switch_Signal
- sheet NMOS Switch3 ports: added 5V_Switch_Signal; removed 3.3V_Switch_Signal
- sheet NMOS Switch4 ports: added 5V_Switch_Signal; removed 3.3V_Switch_Signal
- sheet NMOS Switch5 ports: added 5V_Switch_Signal; removed 3.3V_Switch_Signal
- sheet NMOS Switch6 ports: added 5V_Switch_Signal; removed 3.3V_Switch_Signal
- sheet NMOS Switch7 ports: added 5V_Switch_Signal; removed 3.3V_Switch_Signal
- sheet NMOS Switch8 ports: added 5V_Switch_Signal; removed 3.3V_Switch_Signal
- sheet NMOS Switch9 ports: added 5V_Switch_Signal; removed 3.3V_Switch_Signal
- moved on the sheet: J11
